File: hardware/kubisat_power/kubisat_power.kicad_sch (KiCad schematic)
At the start: 78 parts, among them J1 USB_C_Receptacle_PowerOnly_6P, J2 B2B-PH-SM4-TB_LF__SN_, Q1 Si2305, SW1 SW_Wuerth_450301014042, U2 INA3221, U3 LN2220, U4 CN3791, U5 TP4056, U6 DW01A, U7 FS8205

Commit message: more traces
Parts:
- removed SW1: SW_Wuerth_450301014042, Button_Switch_THT:SW_Slide-03_Wuerth-WS-SLTV_10x2.5x6.4_P2.54mm, symbol Switch:SW_Wuerth_450301014042
- added J3: Conn_01x08_MountingPin, Connector_JST:JST_PH_S8B-PH-SM4-TB_1x08-1MP_P2.00mm_Horizontal, symbol Connector_Generic_MountingPin:Conn_01x08_MountingPin
Connections:
- net +3V3: now also J3.3 (Pin_3)
- net +5V: now also R7.1, R8.1, J3.4 (Pin_4); no longer R10.1, R11.2
- net +BATT: now also R10.1, R11.2; no longer R7.1, R8.1
- net 5V_SENSE_IN: now also R6.1, R8.2; no longer R11.1, R9.1
- net GND: now also J3.1 (Pin_1), J3.2 (Pin_2)
- net INA3221_SCL: now also J3.6 (Pin_6)
- net INA3221_SDA: now also J3.5 (Pin_5)
- net SOLAR_SENSE_IN: now also R11.1, R9.1; no longer R3.1, R5.1
- net USB_SENSE_IN: now also R3.1, R5.1; no longer R6.1, R8.2
Other:
- moved on the sheet: JP1

Commit message: complete routing, changed usb and side terminal - this version was ordered in jlcpcb
Parts:
- removed J3: Conn_01x08_MountingPin, Connector_JST:JST_PH_S8B-PH-SM4-TB_1x08-1MP_P2.00mm_Horizontal, symbol Connector_Generic_MountingPin:Conn_01x08_MountingPin
- added H1, H2, H3, H4: MountingHole, MountingHole:MountingHole_3.2mm_M3_DIN965, symbol Mechanical:MountingHole
- added J3: Conn_01x06_MountingPin, Connector_JST:JST_PH_S6B-PH-SM4-TB_1x06-1MP_P2.00mm_Horizontal, symbol Connector_Generic_MountingPin:Conn_01x06_MountingPin
- J1: footprint Connector_USB:USB_C_Receptacle_HRO_TYPE-C-31-M-17 -> Connector_USB:GCT_USB4140-GF-0230-C_REV0.4
Connections:
- net +3V3: now also J3.3 (Pin_3)
- net +5V: now also J3.4 (Pin_4)
- net GND: now also J1.S1 (SHIELD), J3.1 (Pin_1), J3.2 (Pin_2)
- net INA3221_SCL: now also J3.6 (Pin_6)
- net INA3221_SDA: now also J3.5 (Pin_5)
