File: hardware/kubisat_main/gps.kicad_sch (KiCad schematic)
At the start: 0 parts

Commit message: added arduino code, more items on main schematic
Parts:
- added BT1: Battery_Cell, Battery:BatteryHolder_Seiko_MS621F, symbol Device:Battery_Cell
- added C1: 220u/10V, Capacitor_Tantalum_SMD:CP_EIA-6032-15_Kemet-U, symbol Device:C_Polarized
- added C2: 100n, Capacitor_SMD:C_0805_2012Metric, symbol Device:C
- added D1: 1N5817, Diode_SMD:D_SOD-123, symbol Device:D_Schottky
- added J1: IPX, Connector_Coaxial:U.FL_Hirose_U.FL-R-SMT-1_Vertical, symbol Connector:Conn_Coaxial_Small
- added L1: 27uH, Inductor_SMD:L_0805_2012Metric, symbol Device:L
- added R1: 22, Resistor_SMD:R_0805_2012Metric, symbol Device:R
- added R2: 1k, Resistor_SMD:R_0805_2012Metric, symbol Device:R
- added U2: NEO-6M-GPS, RF_GPS:XCVR_NEO-6M-GPS, symbol RF_GPS:NEO-6M-GPS
Connections:
- new net: L1.1, R1.2
- new net: BT1.1 (+), R2.2, U2.22 (V_BCKP)
- new net: R1.1, U2.8 (RSVD_8), U2.9 (VCC_RF)
- new net: D1.1 (K), R2.1
- new net +3V3: C1.1, C2.1, D1.2 (A), U2.23 (VCC)
- new net GND: BT1.2 (-), C1.2, C2.2, J1.2 (Ext), U2.10 (GND), U2.12 (GND), U2.13 (GND), U2.24 (GND), U2.7 (VDDUSB)
- new net RF_IN: J1.1 (In), L1.2, U2.11 (RF_IN)
Other:
- note added: "ublox NEO-6M-0"

Commit message: added elements and traces to main pcb
Parts:
- U2: footprint RF_GPS:XCVR_NEO-6M-GPS -> NEO-6M-GPS:XCVR_NEO-6M-GPS
Changed lines of the file:
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@@
 			)
 		)
-		(property "Footprint" "RF_GPS:XCVR_NEO-6M-GPS"
+		(property "Footprint" "NEO-6M-GPS:XCVR_NEO-6M-GPS"
 			(at 76.2 121.92 0)
 			(effects

Commit message: added microsd footprint
Parts:
- added U5: XL1278-SMT, RF:XL1278-SMT, symbol RF:XL1278-SMT
Changed lines of the file:
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@@
+	)
+	(symbol
+		(lib_id "RF:XL1278-SMT")
+		(at 231.14 95.25 0)
+		(unit 1)
+		(exclude_from_sim no)
+		(in_bom yes)
+		(on_board yes)
+		(dnp no)
+		(fields_autoplaced yes)
+		(property "Reference" "U5"
+			(at 231.14 66.04 0)
+			(effects
+				(font
+					(size 1.27 1.27)
+				)
+			)
+		)
+		(property "Value" "XL1278-SMT"
+			(at 231.14 68.58 0)
+			(effects
+				(font
+					(size 1.27 1.27)
+				)
+			)
+		)
+		(property "Footprint" "RF:XL1278-SMT"
+			(at 231.14 95.25 0)
+			(effects
+				(font
+					(size 1.27 1.27)
+				)
+				(hide yes)
+			)
+		)
+		(property "Datasheet" ""
+			(at 231.14 95.25 0)
+			(effects
+				(font
+					(size 1.27 1.27)
+				)
+				(hide yes)
+			)
+		)
+		(property "Description" ""
+			(at 231.14 95.25 0)
+			(effects
+				(font
+					(size 1.27 1.27)
+				)
+				(hide yes)
+			)
+		)
+		(pin "15"
+		)
+		(pin "6"
+		)
+		(pin "14"
+		)
+		(pin "4"
+		)
+		(pin "7"
+		)
+		(pin "8"
+		)
+		(pin "5"
+		)
+		(pin "12"
+		)
+		(pin "3"
+		)
+		(pin "16"
+		)
+		(pin "9"
+		)
+		(pin "13"
+		)
+		(pin "10"
+		)
+		(pin "1"
+		)
+		(pin "11"
+		)
+		(pin "2"
+		)
+		(instances
+			(project "kubisat_main"
+				(path "/8e012760-7134-459b-b212-1cb69dd2e1ec/30e74b89-024d-46d7-9097-1329f2d05fbe"
+					(reference "U5")
+					(unit 1)
+				)
+			)
+		)
 	)
 	(symbol
