File: hardware/kubisat_main/comms_protection.kicad_sch (KiCad schematic)
At the start: 0 parts

Commit message: added pcb elements
Parts:
- added J3: POWER_IN, Connector_JST:JST_PH_S6B-PH-SM4-TB_1x06-1MP_P2.00mm_Horizontal, symbol Connector_Generic_MountingPin:Conn_01x06_MountingPin
- added Q1, Q2: BSS138, Package_TO_SOT_SMD:SOT-23, symbol Transistor_FET:BSS138
- added R16, R17, R18, R19: 10k, symbol Device:R
Connections:
- new net 3V3: Q1.1 (G), Q2.1 (G), R17.1, R19.1
- new net 5VIN: J3.4 (Pin_4), R16.1, R18.1
- new net GND: J3.1 (Pin_1), J3.2 (Pin_2), J3.MP (MountPin)
- new net I2C0_SCL: J3.6 (Pin_6), Q1.2 (S), Q1.3 (D), R16.2, R17.2
- new net I2C0_SDA: J3.5 (Pin_5), Q2.2 (S), Q2.3 (D), R18.2, R19.2
- new net NC: J3.3 (Pin_3)
Other:
- note added: "LEVEL_SHIFTER"
