File: hardware/kubisat_main/kubisat_main.kicad_pcb (KiCad board)
At the start: 2 copper layers, 80 x 80 mm, 38 parts, among them J1 DEBUG_SWD, J2 Micro_SD_Card_Det1, J3 UART0, J4 POWER_IN, J5 IPX, J6 POWER, J7 I2C1, J8 SPI0, Q1 BSS138, Q2 BSS138, SW2 RESET, U1 DS3231M, U3 NEO-6M-GPS, U4 XL1278-SMT, U6 Pico

Commit message: finished main board
Parts:
- removed C17: 220u/10V, Capacitor_Tantalum_SMD:CP_EIA-6032-15_Kemet-U
- J1, J3: footprint Connector_PinHeader_1.00mm:PinHeader_1x03_P1.00mm_Vertical -> Connector_PinHeader_2.54mm:PinHeader_1x03_P2.54mm_Horizontal; moved to B.Cu
- J6: footprint Connector_JST:JST_PH_B3B-PH-SM4-TB_1x03-1MP_P2.00mm_Vertical -> Connector_JST:JST_PH_S3B-PH-SM4-TB_1x03-1MP_P2.00mm_Horizontal
- J7: footprint Connector_JST:JST_PH_B2B-PH-SM4-TB_1x02-1MP_P2.00mm_Vertical -> Connector_JST:JST_PH_S2B-PH-SM4-TB_1x02-1MP_P2.00mm_Horizontal; moved to B.Cu
- J8: footprint Connector_JST:JST_PH_B4B-PH-SM4-TB_1x04-1MP_P2.00mm_Vertical -> Connector_JST:JST_PH_S4B-PH-SM4-TB_1x04-1MP_P2.00mm_Horizontal; moved to B.Cu
- SW2: footprint Button_Switch_SMD:SW_SPST_B3SL-1002P -> Button_Switch_SMD:SW_Push_1P1T_NO_CK_KMR2
- moved J1 73.3 mm to (34.4, 69.6), turned to -90 degrees
- moved J3 63.9 mm to (43.7, 69.7), turned to -90 degrees
- moved J5 33.7 mm to (45.4, 111.6), turned to -90 degrees
- moved C2 25.2 mm to (38.4, 84.7), turned to 90 degrees
- moved L1 23.7 mm to (44.2, 108.0)
- moved J7 22.4 mm to (68.3, 91.5), turned to 180 degrees
- moved J8 20.8 mm to (56.4, 91.5), turned to 180 degrees
- moved R11 20.7 mm to (40.2, 108.0)
- moved U3 19.3 mm to (39.4, 98.8), turned to 90 degrees
- moved C16 17.1 mm to (40.7, 89.3)
- moved C1 15.3 mm to (47.2, 84.7), turned to 90 degrees
- moved JP1 14.8 mm to (44.8, 89.5)
- moved R1 11.5 mm to (72.1, 65.3), turned to 180 degrees
- moved R2 11.5 mm to (72.0, 67.5), turned to 180 degrees
- moved J6 11.4 mm to (56.0, 107.7)
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Connections:
- C16 pad 1: +3V3 -> 3V3_GPS
- J2 pad 2: /CS -> SD.CS
- J2 pad 3: /MOSI -> SD.MOSI
- J2 pad 5: /CLK -> SD.CLK
- J2 pad 7: /MISO -> SD.MISO
- R3 pad 2: /CS -> SD.CS
- R4 pad 2: /MOSI -> SD.MOSI
- R5 pad 2: /CLK -> SD.CLK
- R6 pad 2: /MISO -> SD.MISO
- SW2 pad 1: Net-(SW2-Pad1) -> GND
- U4 pad 10: /DIO0 -> SX1278.DIO0
- U4 pad 11: /RES -> SX1278.RES
- U4 pad 2: /DIO1 -> SX1278.DIO1
- U4 pad 6: /MISO -> SX1278.MISO
- U4 pad 7: /MOSI -> SX1278.MOSI
- U4 pad 8: /SCLK -> SX1278.SCLK
- U4 pad 9: /NSS -> SX1278.NSS
- U6 pad 13: unconnected-(U6-GND-Pad13) -> GND
- U6 pad 18: unconnected-(U6-GND-Pad18) -> GND
- U6 pad 23: unconnected-(U6-GND-Pad23) -> GND
- U6 pad 28: SX1278.GND -> GND
- U6 pad 38: Net-(SW2-Pad1) -> GND
- U6 pad 8: unconnected-(U6-GND-Pad8) -> GND
Routing:
- net GND: track 0.00 -> 582.3 mm, vias 0 -> 13
- net +5V: track 0.00 -> 186.0 mm, vias 0 -> 8
- net Net-(J1-Pin_1): track 0.00 -> 106.6 mm, vias 0 -> 1
- net 3V_BACKUP: track 0.00 -> 105.9 mm, vias 0 -> 2
- net Net-(J1-Pin_3): track 0.00 -> 104.8 mm, vias 0 -> 1
- net SPI0_SCK: track 0.00 -> 84.6 mm, vias 0 -> 3
- net SPI0_CS: track 0.00 -> 81.8 mm, vias 0 -> 3
- net +3.3V: track 0.00 -> 80.6 mm, vias 0 -> 4
- net SPI0_MISO: track 0.00 -> 73.0 mm, vias 0 -> 3
- net GPS_RX: track 0.00 -> 70.1 mm
- net SPI0_MOSI: track 0.00 -> 69.9 mm, vias 0 -> 1
- net I2C1_SCL: track 0.00 -> 69.2 mm, vias 0 -> 3
- net GPS_TX: track 0.00 -> 66.9 mm
- net I2C1_SDA: track 0.00 -> 65.4 mm, vias 0 -> 3
- net Net-(J3-Pin_1): track 0.00 -> 59.4 mm, vias 0 -> 1
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Other:
- board text added: "CS"
- board text added: "DEBUG"
- board text added: "DS3231"
- board text added: "GND"
- board text added: "GND GND NC +5V SDA SCL"
- board text added: "GND SENSOR_EN +5V"
- board text added: "I2C1"
- board text added: "KUBISAT V1 2024"
- board text added: "Labor omnia vincit"
- board text added: "MICRO_SD"
- board text added: "MISO"
- board text added: "MOSI"
- board text added: "POWER_IN"
- board text added: "POWER_OUT"
- board text added: "RPI PICO"
- board text added: "RXD"
- board text added: "SCK"
- board text added: "SCL"
- board text added: "SDA"
- board text added: "SPI0"
- board text added: "SWCLK"
- board text added: "SWDIO"
- board text added: "SX1278"
- board text added: "TXD"
- board text added: "UART0"
