File: hardware/kubisat_sensor/kubisat_sensors/kubisat_sensors.kicad_sch (KiCad schematic)
At the start: 19 parts, among them U1 MPU-6050, U2 BME280, U3 MMC5883MA, U4 DS3231M

Commit message: changed folder structure
Parts:
- removed C1, C2, C5: 100n, Capacitor_SMD:C_0805_2012Metric, symbol Device:C
- removed C3: 2n2, Capacitor_SMD:C_0805_2012Metric, symbol Device:C
- removed C4: 10n, Capacitor_SMD:C_0805_2012Metric, symbol Device:C
- removed C6: 1u, Capacitor_SMD:C_0805_2012Metric, symbol Device:C
- removed C7: 4u7, Capacitor_SMD:C_0805_2012Metric, symbol Device:C
- removed C8: 200n, Capacitor_SMD:C_0805_2012Metric, symbol Device:C
- removed R1, R3, R5, R7: 10k, Resistor_SMD:R_0805_2012Metric, symbol Device:R
- removed R2, R4, R6: 4k7, Resistor_SMD:R_0805_2012Metric, symbol Device:R
- removed U1: MPU-6050, Sensor_Motion:InvenSense_QFN-24_4x4mm_P0.5mm, symbol Sensor_Motion:MPU-6050
- removed U2: BME280, Package_LGA:Bosch_LGA-8_2.5x2.5mm_P0.65mm_ClockwisePinNumbering, symbol Sensor:BME280
- removed U3: MMC5883MA, Package_LGA:LGA-16_3x3mm_P0.5mm, symbol Sensor_Magnetic:MMC5883MA
- removed U4: DS3231M, Package_SO:SOIC-16W_7.5x10.3mm_P1.27mm, symbol Timer_RTC:DS3231M
Other:
- note removed: "9DOF MPU6050 + HMC5883L"
- note removed: "BMP280 I2C MODE"

Commit message: added sensors board
Parts:
- added C1, C2: 10u, Capacitor_Tantalum_SMD:CP_EIA-3216-18_Kemet-A, symbol Device:C_Polarized
- added J1: POWER, Connector_JST:JST_PH_S3B-PH-SM4-TB_1x03-1MP_P2.00mm_Horizontal, symbol Connector_Generic_MountingPin:Conn_01x03_MountingPin
- added J2: I2C1, Connector_JST:JST_PH_S2B-PH-SM4-TB_1x02-1MP_P2.00mm_Horizontal, symbol Connector_Generic_MountingPin:Conn_01x02_MountingPin
- added J3, J4, J5, J8: Conn_01x08, Connector_PinSocket_2.54mm:PinSocket_1x08_P2.54mm_Vertical, symbol Connector_Generic:Conn_01x08
- added J7: SPI0, Connector_JST:JST_PH_S4B-PH-SM4-TB_1x04-1MP_P2.00mm_Horizontal, symbol Connector_Generic_MountingPin:Conn_01x04_MountingPin
- added U1: ~, Package_TO_SOT_SMD:SOT-23-5, symbol kubisat1:LDI8119-3.3EN
Connections:
- new net +3V3: C2.1, J3.1 (Pin_1), J4.1 (Pin_1), J5.1 (Pin_1), J8.1 (Pin_1), U1.5 (VOUT)
- new net +5V: C1.1, J1.3 (Pin_3), U1.1 (VIN)
- new net GND: C1.2, C2.2, J1.1 (Pin_1), J1.MP (MountPin), J2.MP (MountPin), J3.2 (Pin_2), J4.2 (Pin_2), J5.2 (Pin_2), J7.MP (MountPin), J8.2 (Pin_2), U1.2 (GND)
- new net SENSOR_POWER_ENABLE: J1.2 (Pin_2), U1.3 (EN)
- new net SENSOR_SCL: J2.2 (Pin_2), J3.3 (Pin_3), J4.3 (Pin_3), J5.3 (Pin_3), J7.4 (Pin_4), J8.3 (Pin_3)
- new net SENSOR_SDA: J2.1 (Pin_1), J3.4 (Pin_4), J4.4 (Pin_4), J5.4 (Pin_4), J7.3 (Pin_3), J8.4 (Pin_4)
